Commit message: feat: add collion detection support + unit tests

File: source/robot_model/test/fixtures/ur5e.urdf (robot description, URDF)
Before this commit: robot ur, 11 links, 10 joints
Links:
- link ur5e_base_link_inertia: geometry collision mesh filename=/src/source/robot_model/test/fixtures/ur5e/collision/base.s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; visual mesh filename=/src/source/robot_model/test/fixtures/ur5e/visual/base.dae
- link ur5e_forearm_link: geometry collision mesh filename=/src/source/robot_model/test/fixtures/ur5e/collision/forear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; visual mesh filename=/src/source/robot_model/test/fixtures/ur5e/visual/forearm.d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
- link ur5e_shoulder_link: geometry collision mesh filename=/src/source/robot_model/test/fixtures/ur5e/collision/should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; visual mesh filename=/src/source/robot_model/test/fixtures/ur5e/visual/shoulder.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
- link ur5e_upper_arm_link: geometry collision mesh filename=/src/source/robot_model/test/fixtures/ur5e/collision/uppera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; visual mesh filename=/src/source/robot_model/test/fixtures/ur5e/visual/upperarm.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
- link ur5e_wrist_1_link: geometry collision mesh filename=/src/source/robot_model/test/fixtures/ur5e/collision/wrist1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; visual mesh filename=/src/source/robot_model/test/fixtures/ur5e/visual/wrist1.dae
- link ur5e_wrist_2_link: geometry collision mesh filename=/src/source/robot_model/test/fixtures/ur5e/collision/wrist2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; visual mesh filename=/src/source/robot_model/test/fixtures/ur5e/visual/wrist2.dae
- link ur5e_wrist_3_link: geometry collision mesh filename=/src/source/robot_model/test/fixtures/ur5e/collision/wrist3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; visual mesh filename=/src/source/robot_model/test/fixtures/ur5e/visual/wrist3.dae

Commit message: Revert "feat: integrate collision detection feature into robot model (#163)"
This reverts commit 852f16400c8d688ef5e91142034e3b9c3cabe5e0.

File: source/robot_model/test/fixtures/ur5e.urdf (robot description, URDF)
Before this commit: robot ur5e, 13 links, 12 joints
Links:
- removed link ur5e_base_link
- removed link ur5e_ft_frame
Joints:
- removed joint ur5e_base_joint
- removed joint ur5e_wrist_3_link-ft_frame
- joint ur5e_base_link-base_fixed_joint: parent ur5e_base_link -> world
- joint ur5e_base_link-base_link_inertia: parent ur5e_base_link -> world
